File: 4to16rowFets.sch (KiCad schematic (older format))
At the start: 26 parts, among them M301 FDS4935BZ, M302 FDS4935BZ, M303 FDS4935BZ, M304 FDS4935BZ, M305 FDS4935BZ, M306 FDS4935BZ, M307 FDS4935BZ, M308 FDS4935BZ, U301 74154

Commit message: Improved connector placement
Changed lines of the file:
@@
 $Descr A4 11693 8268
 encoding utf-8
-Sheet 6 7
+Sheet 4 7
 Title ""
 Date ""
@@
 AR Path="/5713FA0A/5716BBBF/5713FCB1" Ref="U401"  Part="1"
 AR Path="/5713FA0A/5716C198/5713FCB1" Ref="U501"  Part="1"
-F 0 "U601" H 2200 2816 50  0000 C CNN
+F 0 "U301" H 2200 2816 50  0000 C CNN
 F 1 "74154" H 2200 2725 50  0000 C CNN
 F 2 "Housings_SOIC:SOIC-24_7.5x15.4mm_Pitch1.27mm" H 2200 1700 60  0001 C CNN
@@
 AR Path="/5713FA0A/5716BBBF/57140FE8" Ref="C401"  Part="1"
 AR Path="/5713FA0A/5716C198/57140FE8" Ref="C501"  Part="1"
-F 0 "C601" H 1465 2196 50  0000 L CNN
+F 0 "C301" H 1465 2196 50  0000 L CNN
 F 1 "0.1uF" H 1465 2105 50  0000 L CNN
 F 2 "Capacitors_SMD:C_0603_HandSoldering" H 1388 2000 50  0001 C CNN
@@
 AR Path="/5713FA0A/5716C198/57141250" Ref="M501"  Part="1"
 AR Path="/5713FA0A/5716B5E6/57141250" Ref="M601"  Part="1"
-F 0 "M601" H 4350 3300 50  0000 C CNN
+F 0 "M301" H 4350 3300 50  0000 C CNN
 F 1 "FDS4935BZ" H 4500 2000 50  0000 C CNN
 F 2 "Housings_SOIC:SOIC-8_3.9x4.9mm_Pitch1.27mm" H 4600 2700 20  0001 C CNN
@@
 AR Path="/5713FA0A/5716C198/57142A13" Ref="M502"  Part="1"
 AR Path="/5713FA0A/5716B5E6/57142A13" Ref="M602"  Part="1"
-F 0 "M602" H 6400 3415 50  0000 C CNN
+F 0 "M302" H 6400 3415 50  0000 C CNN
 F 1 "FDS4935BZ" H 6400 3324 50  0000 C CNN
 F 2 "Housings_SOIC:SOIC-8_3.9x4.9mm_Pitch1.27mm" H 6400 2700 20  0001 C CNN
@@
 AR Path="/5713FA0A/5716C198/57142D25" Ref="M504"  Part="1"
 AR Path="/5713FA0A/5716B5E6/57142D25" Ref="M604"  Part="1"
-F 0 "M604" H 10000 3415 50  0000 C CNN
+F 0 "M304" H 10000 3415 50  0000 C CNN
 F 1 "FDS4935BZ" H 10000 3324 50  0000 C CNN
 F 2 "Housings_SOIC:SOIC-8_3.9x4.9mm_Pitch1.27mm" H 10000 2700 20  0001 C CNN
@@
 AR Path="/5713FA0A/5716C198/57142D6E" Ref="M506"  Part="1"
 AR Path="/5713FA0A/5716B5E6/57142D6E" Ref="M606"  Part="1"
-F 0 "M606" H 6400 5965 50  0000 C CNN
+F 0 "M306" H 6400 5965 50  0000 C CNN
 F 1 "FDS4935BZ" H 6400 5874 50  0000 C CNN
 F 2 "Housings_SOIC:SOIC-8_3.9x4.9mm_Pitch1.27mm" H 6400 5250 20  0001 C CNN
@@
 AR Path="/5713FA0A/5716C198/57143035" Ref="M507"  Part="1"
 AR Path="/5713FA0A/5716B5E6/57143035" Ref="M607"  Part="1"
-F 0 "M607" H 8200 5965 50  0000 C CNN
+F 0 "M307" H 8200 5965 50  0000 C CNN
 F 1 "FDS4935BZ" H 8200 5874 50  0000 C CNN
 F 2 "Housings_SOIC:SOIC-8_3.9x4.9mm_Pitch1.27mm" H 8200 5250 20  0001 C CNN
@@
 AR Path="/5713FA0A/5716C198/57143083" Ref="M508"  Part="1"
 AR Path="/5713FA0A/5716B5E6/57143083" Ref="M608"  Part="1"
-F 0 "M608" H 10000 5965 50  0000 C CNN
+F 0 "M308" H 10000 5965 50  0000 C CNN
 F 1 "FDS4935BZ" H 10000 5874 50  0000 C CNN
 F 2 "Housings_SOIC:SOIC-8_3.9x4.9mm_Pitch1.27mm" H 10000 5250 20  0001 C CNN
@@
 AR Path="/5713FA0A/5716BBBF/571445D8" Ref="PAD401"  Part="1"
 AR Path="/5713FA0A/5716C198/571445D8" Ref="PAD501"  Part="1"
-F 0 "PAD601" H 5050 2250 50  0000 C CNN
+F 0 "PAD301" H 5050 2250 50  0000 C CNN
 F 1 "2_54_1_0" H 5100 2150 50  0000 C CNN
 F 2 "Wire_Pads:wirepad-2_54_1_0" H 5230 2400 20  0001 C CNN
@@
 AR Path="/5713FA0A/5716BBBF/57144DD0" Ref="PAD409"  Part="1"
 AR Path="/5713FA0A/5716C198/57144DD0" Ref="PAD509"  Part="1"
-F 0 "PAD609" H 5050 2850 50  0000 C CNN
+F 0 "PAD309" H 5050 2850 50  0000 C CNN
 F 1 "2_54_1_0" H 5100 2750 50  0000 C CNN
 F 2 "Wire_Pads:wirepad-2_54_1_0" H 5230 3000 20  0001 C CNN
@@
 AR Path="/5713FA0A/5716BBBF/57144F5E" Ref="PAD417"  Part="1"
 AR Path="/5713FA0A/5716C198/57144F5E" Ref="PAD517"  Part="1"
-F 0 "PAD617" H 5050 4800 50  0000 C CNN
+F 0 "PAD317" H 5050 4800 50  0000 C CNN
 F 1 "2_54_1_0" H 5100 4700 50  0000 C CNN
 F 2 "Wire_Pads:wirepad-2_54_1_0" H 5230 4950 20  0001 C CNN
@@
 AR Path="/5713FA0A/5716BBBF/57144F6A" Ref="PAD425"  Part="1"
 AR Path="/5713FA0A/5716C198/57144F6A" Ref="PAD525"  Part="1"
-F 0 "PAD625" H 5050 5400 50  0000 C CNN
+F 0 "PAD325" H 5050 5400 50  0000 C CNN
 F 1 "2_54_1_0" H 5100 5300 50  0000 C CNN
 F 2 "Wire_Pads:wirepad-2_54_1_0" H 5230 5550 20  0001 C CNN
@@
 AR Path="/5713FA0A/5716BBBF/57145146" Ref="PAD402"  Part="1"
 AR Path="/5713FA0A/5716C198/57145146" Ref="PAD502"  Part="1"
-F 0 "PAD602" H 6850 2250 50  0000 C CNN
+F 0 "PAD302" H 6850 2250 50  0000 C CNN
 F 1 "2_54_1_0" H 6900 2150 50  0000 C CNN
 F 2 "Wire_Pads:wirepad-2_54_1_0" H 7030 2400 20  0001 C CNN
@@
 AR Path="/5713FA0A/5716BBBF/57145154" Ref="PAD410"  Part="1"
 AR Path="/5713FA0A/5716C198/57145154" Ref="PAD510"  Part="1"
-F 0 "PAD610" H 6850 2850 50  0000 C CNN
+F 0 "PAD310" H 6850 2850 50  0000 C CNN
 F 1 "2_54_1_0" H 6900 2750 50  0000 C CNN
 F 2 "Wire_Pads:wirepad-2_54_1_0" H 7030 3000 20  0001 C CNN
@@
 AR Path="/5713FA0A/5716BBBF/57145162" Ref="PAD418"  Part="1"
 AR Path="/5713FA0A/5716C198/57145162" Ref="PAD518"  Part="1"
-F 0 "PAD618" H 6850 4800 50  0000 C CNN
+F 0 "PAD318" H 6850 4800 50  0000 C CNN
 F 1 "2_54_1_0" H 6900 4700 50  0000 C CNN
 F 2 "Wire_Pads:wirepad-2_54_1_0" H 7030 4950 20  0001 C CNN
@@
 AR Path="/5713FA0A/5716BBBF/57145170" Ref="PAD426"  Part="1"
 AR Path="/5713FA0A/5716C198/57145170" Ref="PAD526"  Part="1"
-F 0 "PAD626" H 6850 5400 50  0000 C CNN
+F 0 "PAD326" H 6850 5400 50  0000 C CNN
 F 1 "2_54_1_0" H 6900 5300 50  0000 C CNN
 F 2 "Wire_Pads:wirepad-2_54_1_0" H 7030 5550 20  0001 C CNN
@@
 AR Path="/5713FA0A/5716BBBF/571452E2" Ref="PAD403"  Part="1"
 AR Path="/5713FA0A/5716C198/571452E2" Ref="PAD503"  Part="1"
-F 0 "PAD603" H 8650 2250 50  0000 C CNN
+F 0 "PAD303" H 8650 2250 50  0000 C CNN
 F 1 "2_54_1_0" H 8700 2150 50  0000 C CNN
 F 2 "Wire_Pads:wirepad-2_54_1_0" H 8830 2400 20  0001 C CNN
@@
 AR Path="/5713FA0A/5716BBBF/571452F0" Ref="PAD411"  Part="1"
 AR Path="/5713FA0A/5716C198/571452F0" Ref="PAD511"  Part="1"
-F 0 "PAD611" H 8650 2850 50  0000 C CNN
+F 0 "PAD311" H 8650 2850 50  0000 C CNN
 F 1 "2_54_1_0" H 8700 2750 50  0000 C CNN
 F 2 "Wire_Pads:wirepad-2_54_1_0" H 8830 3000 20  0001 C CNN
@@
 AR Path="/5713FA0A/5716BBBF/571452FE" Ref="PAD419"  Part="1"
 AR Path="/5713FA0A/5716C198/571452FE" Ref="PAD519"  Part="1"
-F 0 "PAD619" H 8650 4800 50  0000 C CNN
+F 0 "PAD319" H 8650 4800 50  0000 C CNN
 F 1 "2_54_1_0" H 8700 4700 50  0000 C CNN
 F 2 "Wire_Pads:wirepad-2_54_1_0" H 8830 4950 20  0001 C CNN
@@
 AR Path="/5713FA0A/5716BBBF/5714530C" Ref="PAD427"  Part="1"
 AR Path="/5713FA0A/5716C198/5714530C" Ref="PAD527"  Part="1"
-F 0 "PAD627" H 8650 5400 50  0000 C CNN
+F 0 "PAD327" H 8650 5400 50  0000 C CNN
 F 1 "2_54_1_0" H 8700 5300 50  0000 C CNN
 F 2 "Wire_Pads:wirepad-2_54_1_0" H 8830 5550 20  0001 C CNN
@@
 AR Path="/5713FA0A/5716BBBF/5714549E" Ref="PAD404"  Part="1"
 AR Path="/5713FA0A/5716C198/5714549E" Ref="PAD504"  Part="1"
-F 0 "PAD604" H 10450 2250 50  0000 C CNN
+F 0 "PAD304" H 10450 2250 50  0000 C CNN
 F 1 "2_54_1_0" H 10500 2150 50  0000 C CNN
 F 2 "Wire_Pads:wirepad-2_54_1_0" H 10630 2400 20  0001 C CNN
@@
 AR Path="/5713FA0A/5716BBBF/571454AC" Ref="PAD412"  Part="1"
 AR Path="/5713FA0A/5716C198/571454AC" Ref="PAD512"  Part="1"
-F 0 "PAD612" H 10450 2850 50  0000 C CNN
+F 0 "PAD312" H 10450 2850 50  0000 C CNN
 F 1 "2_54_1_0" H 10500 2750 50  0000 C CNN
 F 2 "Wire_Pads:wirepad-2_54_1_0" H 10630 3000 20  0001 C CNN
@@
 AR Path="/5713FA0A/5716BBBF/571454BA" Ref="PAD420"  Part="1"
 AR Path="/5713FA0A/5716C198/571454BA" Ref="PAD520"  Part="1"
-F 0 "PAD620" H 10450 4800 50  0000 C CNN
+F 0 "PAD320" H 10450 4800 50  0000 C CNN
 F 1 "2_54_1_0" H 10500 4700 50  0000 C CNN
 F 2 "Wire_Pads:wirepad-2_54_1_0" H 10630 4950 20  0001 C CNN
@@
 AR Path="/5713FA0A/5716BBBF/571454C8" Ref="PAD428"  Part="1"
 AR Path="/5713FA0A/5716C198/571454C8" Ref="PAD528"  Part="1"
-F 0 "PAD628" H 10450 5400 50  0000 C CNN
+F 0 "PAD328" H 10450 5400 50  0000 C CNN
 F 1 "2_54_1_0" H 10500 5300 50  0000 C CNN
 F 2 "Wire_Pads:wirepad-2_54_1_0" H 10630 5550 20  0001 C CNN
@@
 AR Path="/5713FA0A/5716C198/57142EE6" Ref="M505"  Part="1"
 AR Path="/5713FA0A/5716B5E6/57142EE6" Ref="M605"  Part="1"
-F 0 "M605" H 4600 5965 50  0000 C CNN
+F 0 "M305" H 4600 5965 50  0000 C CNN
 F 1 "FDS4935BZ" H 4600 5874 50  0000 C CNN
 F 2 "Housings_SOIC:SOIC-8_3.9x4.9mm_Pitch1.27mm" H 4600 5250 20  0001 C CNN
@@
 AR Path="/5713FA0A/5716C198/57142CD2" Ref="M503"  Part="1"
 AR Path="/5713FA0A/5716B5E6/57142CD2" Ref="M603"  Part="1"
-F 0 "M603" H 8200 3415 50  0000 C CNN
+F 0 "M303" H 8200 3415 50  0000 C CNN
 F 1 "FDS4935BZ" H 8200 3324 50  0000 C CNN
 F 2 "Housings_SOIC:SOIC-8_3.9x4.9mm_Pitch1.27mm" H 8200 2700 20  0001 C CNN
